Commit message: ros2 sim

File: src/ros2_dream_base_description/urdf/diff_drive.gazebo.xacro (robot description, xacro)
@@ -2,6 +2,6 @@
 <robot name="dream_gazebo_diff_drive" xmlns:xacro="http://www.ros.org/wiki/xacro">
     <!-- Notes: load urdf, then load diff params -->
-    <xacro:include filename="$(find dream_base_description)/urdf/diff_drive.urdf.xacro" />
-    <xacro:property name="diff_params" value="${load_yaml('$(find dream_base_description)/config/diff_params.yaml')}" />`
+    <xacro:include filename="$(find ros2_dream_base_description)/urdf/diff_drive.urdf.xacro" />
+    <xacro:property name="diff_params" value="${xacro.load_yaml('$(find ros2_dream_base_description)/config/diff_params.yaml')}" />`
     <gazebo>
         <!-- Notes: use params loaded from yaml -->

File: src/ros2_dream_base_description/urdf/diff_drive.urdf.xacro (robot description, xacro)
@@ -1,5 +1,5 @@
 <?xml version="1.0"?>
 <robot xmlns:xacro="http://www.ros.org/wiki/xacro" name="diff_drive">
-    <xacro:property name="diff_params" value="${load_yaml('$(find dream_base_description)/config/diff_params.yaml')}" />
+    <xacro:property name="diff_params" value="${xacro.load_yaml('$(find ros2_dream_base_description)/config/diff_params.yaml')}" />
     <xacro:property name="grey_mat">
      <material name="arm_grey_mat">
